File: bioptics-bx4x4-dc44-camera-board.kicad_sch (KiCad schematic)
At the start: 21 parts

Commit message: Add USB HS and bipolar analog power supply
Parts:
- added C232, C46, C47, C50, C52, C55, C59, C60, C61, C62, C63, C64, C65, C67, C68, C69, C71, C72: 100nF, Capacitor_SMD:C_0402_1005Metric, symbol Device:C_Small
- added C43: 1nF, Capacitor_SMD:C_1206_3216Metric, symbol Device:C_Small
- added C44: 22uF, Capacitor_SMD:C_0603_1608Metric, symbol Device:C_Small
- added C45, C66, C88: 1uF, Capacitor_SMD:C_0402_1005Metric, symbol Device:C_Small
- added C48, C51, C53, C57, C58: 10uF, Capacitor_SMD:C_0805_2012Metric, symbol Device:C_Small
- added C49: 10uF, Capacitor_Tantalum_SMD:CP_EIA-3216-10_Kemet-I, symbol Device:C_Polarized_Small
- added C54, C56: 20pF, Capacitor_SMD:C_0402_1005Metric, symbol Device:C_Small
- added C70, C73, C74: 4.7uF, Capacitor_SMD:C_0402_1005Metric, symbol Device:C_Small
- added D1, D2, D3: B5819W, Diode_SMD:D_SOD-123, symbol Device:D_Schottky
- added FB8: 600R@100MHz, Inductor_SMD:L_0805_2012Metric, symbol Device:FerriteBead_Small
- added J3: USB_C_Receptacle_USB2.0, Connector_USB:USB_C_Receptacle_Palconn_UTC16-G, symbol Connector:USB_C_Receptacle_USB2.0
- added J4: TagConnect_TC2030_SWD, Connector:Tag-Connect_TC2030-IDC-NL_2x03_P1.27mm_Vertical, symbol Connector_TagConnect:TagConnect_TC2030_SWD
- added L6: 4.7uH, Inductor_SMD:L_Taiyo-Yuden_MD-3030, symbol Device:L
- added L7, L8: 100uH, Inductor_SMD:L_Taiyo-Yuden_NR-30xx, symbol Device:L_Small
- added L9: 10uH, Inductor_SMD:L_0805_2012Metric, symbol Device:L_Small
- added R110, R18, R19, R23: 5.1k, Resistor_SMD:R_0402_1005Metric, symbol Device:R_Small
- added R16: 200k, Resistor_SMD:R_0805_2012Metric, symbol Device:R_Small
- added R17, R21: 20k, Resistor_SMD:R_0402_1005Metric, symbol Device:R_Small
- added R20: 100k, Resistor_SMD:R_0402_1005Metric, symbol Device:R_Small
- added R22: 10kR, Resistor_SMD:R_0402_1005Metric, symbol Device:R_Small
- added R24: 12k, Resistor_SMD:R_0402_1005Metric, symbol Device:R_Small
- added R26, R27, R28, R29: 33, Resistor_SMD:R_0402_1005Metric, symbol Device:R_Small
- added R30, R31: 4.7k, Resistor_SMD:R_0402_1005Metric, symbol Device:R_Small
- added R32: 100, Resistor_SMD:R_0402_1005Metric, symbol Device:R_Small
- added U10: SRV05-4, Package_TO_SOT_SMD:SOT-23-6, symbol Power_Protection:SRV05-4
- added U12: USB3300-EZK, Package_DFN_QFN:QFN-32-1EP_5x5mm_P0.5mm_EP3.45x3.45mm, symbol Interface_USB:USB3300-EZK
- added U13: AMS1117-3.3, Package_TO_SOT_SMD:SOT-223-3_TabPin2, symbol Regulator_Linear:AMS1117-3.3
- added U9: FP6291, Package_TO_SOT_SMD:SOT-23-6, symbol Regulator_Switching_Feeling:FP6291
- added Y1: 24MHz, Crystal:Crystal_SMD_3225-4Pin_3.2x2.5mm, symbol Device:Crystal_GND24_Small
- gave numbers to parts that had none: 21
Connections:
- net 3v3 is gone; now on net +3V3: C76.1, C78.1, C80.1, C82.1, C83.1, C84.1, C85.1, C86.1, C87.1, C89.1, C90.1, C91.1, C92.1, C93.1, R25.1, U14.171 (PDR_ON)
- net 3v3A is gone; now on net +3.3VA: C77.1, U14.38 (VREF+)
- net GND: now also U11.12 (VSSQ), U11.32 (VSSQ), U11.38 (VSSQ), U11.44 (VSS), U11.46 (VSSQ), U11.52 (VSSQ), U11.58 (VSS), U11.6 (VSSQ), U11.72 (VSS), U11.78 (VSSQ), U11.84 (VSSQ), U11.86 (VSS), U11.9 (VSSQ), U14.102 (VSS), U14.113 (VSS), U14.126 (VSS), U14.135 (VSS), U14.14 (VSS), U14.148 (VSS), U14.158 (VSS), U14.22 (VSS), U14.37 (VSSA), U14.48 (VSS), U14.61 (VSS), U14.71 (VSS), U14.90 (VSS), C232.2, C43.1, C44.2, C45.1, C46.2, C47.2, C49.2, C50.2, C51.1, C52.2, C53.1, C54.1, C55.2, C56.2, C57.1, C58.1, C59.2, C60.2, C61.2, C62.2, C63.2, C64.2, C65.2, C66.1, C67.2, C68.2, C69.2, C70.2, C71.2, C72.2, C73.2, C74.2, C88.2, D1.1 (K), J3.A1 (GND), J3.A12 (GND), J3.B1 (GND), J3.B12 (GND), J4.5 (GND), R110.1, R16.1, R17.1, R18.2, R19.1, R22.2, R24.1, U10.2 (VN), U12.1 (GND), U12.2 (GND), U12.33 (GND), U13.1 (GND), U9.2 (GND), Y1.2, Y1.4
- net MCU_~{RST}: now also J4.3 (~{RESET})
- net ULPI_CK: now also U12.14 (CLKOUT)
- net ULPI_D0: now also U12.24 (DATA0)
- net ULPI_D1: now also U12.23 (DATA1)
- net ULPI_D2: now also U12.22 (DATA2)
- net ULPI_D3: now also U12.21 (DATA3)
- net ULPI_D4: now also U12.20 (DATA4)
- net ULPI_D5: now also U12.19 (DATA5)
- net ULPI_D6: now also U12.18 (DATA6)
- net ULPI_D7: now also U12.17 (DATA7)
- net ULPI_DIR: now also U12.12 (DIR)
- net ULPI_NXT: now also U12.11 (NXT)
- net ULPI_STP: now also U12.13 (STP)
- net +3V3: now reaches U11.1 (VDD)
- net +3V3: now also U11.15 (VDD), U11.29 (VDD), U11.3 (VDDQ), U11.35 (VDDQ), U11.41 (VDDQ), U11.43 (VDD), U11.49 (VDDQ), U11.55 (VDDQ), U11.75 (VDDQ), U11.81 (VDDQ), U14.103 (VDD), U14.114 (VDD33_USB), U14.127 (VDD), U14.136 (VDD), U14.149 (VDD), U14.15 (VDD), U14.159 (VDD), U14.172 (VDD), U14.23 (VDD), U14.36 (VDD), U14.49 (VDD), U14.6 (VBAT), U14.62 (VDD), U14.72 (VDD), U14.82 (VDD), U14.91 (VDD), C46.1, C47.1, C50.1, C52.1, C55.1, C59.1, C60.1, C61.1, C62.1, C63.1, C64.1, C65.1, C67.1, C68.1, C70.1, C71.1, L9.1, R30.1, R31.1, R32.1, U12.16 (VDD3.3), U12.25 (VDD3.3), U12.30 (VDD3.3), U12.31 (REG_EN), U12.6 (VDD3.3), U13.2 (VO)
- net IMAGE_SCK_{3}: now reaches U14.1 (PE2)
- net I2C4_SCL: now reaches U14.100 (PD12)
- net I2C4_SDA: now reaches U14.101 (PD13)
- net IRQ_{2}: now reaches U14.111 (PG7)
- net SLAVE_CLK: now reaches U14.119 (PA8)
- net IRQ_{3}: now reaches U14.12 (PI10)
- net IMAGE_~{FRAME}_{4}: now reaches U14.122 (PA11)
- net IO0_{3}: now reaches U14.123 (PA12)
- net at U14.124 (PA13): now also J4.2 (SWDIO)
- net at U14.137 (PA14): now also J4.4 (SWCLK)
- net IMAGE_SCK_{4}: now reaches U14.145 (PD3)
- net IO1_{3}: now reaches U14.146 (PD4)
- net IMAGE_~{FRAME}_{2}: now reaches U14.147 (PD5)
- net IO1_{4}: now reaches U14.150 (PD6)
- net SPI1_MOSI: now reaches U14.151 (PD7)
- net SPI1_MISO: now reaches U14.152 (PG9)
- net SPI1_NSS: now reaches U14.153 (PG10)
- net SPI1_SCK: now reaches U14.154 (PG11)
- net at U14.155 (PG12): now also R26.2
- net IMAGE_SCK_{2}: now reaches U14.156 (PG13)
- net IMAGE_MOSI_{2}: now reaches U14.157 (PG14)
- net at U14.161 (PB3): now also J4.6 (SWO)
- net I2C_SCL: now reaches U14.164 (PB6)
- net I2C_SCL: now also R30.2
- net I2C_SDA: now reaches U14.165 (PB7)
- net I2C_SDA: now also R31.2
- net IO0_{2}: now reaches U14.2 (PE3)
- net IMAGE_~{FRAME}_{1}: now reaches U14.24 (PF6)
- net IMAGE_SCK_{1}: now reaches U14.25 (PF7)
- net at U14.26 (PF8): now also R27.2
- net IMAGE_MOSI_{1}: now reaches U14.27 (PF9)
- net IO0_{1}: now reaches U14.29 (PH0)
- net IMAGE_~{FRAME}_{3}: now reaches U14.3 (PE4)
- net IRQ_{4}: now reaches U14.33 (PC1)
- net +3.3VA: now reaches U14.39 (VDDA)
- net +3.3VA: now also C74.1, C88.1, L9.2
- net at U14.4 (PE5): now also R29.2
- net IMAGE_MOSI_{3}: now reaches U14.5 (PE6)
- net IO1_{1}: now reaches U14.54 (PC4)
- net IO1_{2}: now reaches U14.55 (PC5)
- net IRQ_{1}: now reaches U14.58 (PB2)
- net IO0_{4}: now reaches U14.8 (PC13)
- net SLAVE_RST: now reaches U14.9 (PC14)
- net at U14.94 (PB14): now also R28.2
- net IMAGE_MOSI_{4}: now reaches U14.95 (PB15)
- new net: C56.1, U12.28 (XI), Y1.1
- new net: C53.2, D3.2 (A), L7.1
- new net: C48.1, D2.2 (A), L6.2, U9.1 (LX)
- new net: C66.2, FB8.1, U13.3 (VI)
- new net: J4.1 (VTGT), R32.2
- new net: J3.A5 (CC1), R18.1
- new net: J3.B5 (CC2), R19.2
- new net: C43.2, J3.S1 (SHIELD), R16.2
- new net: C54.2, U12.27 (XO), Y1.3
- new net: C69.1, C73.1, U12.15 (VDD1.8), U12.26 (VDD1.8)
- new net: C72.1, U12.29 (VDDA1.8)
- new net: R24.2, U12.32 (RBIAS)
- new net: R23.1, U12.4 (VBUS)
- new net: R110.2, U12.9 (RESET)
- new net: C51.2, D2.1 (K), L8.1, R20.1
- new net: R20.2, R21.1
- new net: R21.2, R22.1, U9.3 (FB)
- new net: C48.2, D1.2 (A), D3.1 (K)
- new net: R17.2, U9.6 (OC)
- new net +5V: C232.1, C44.1, C45.2, C49.1, FB8.2, J3.A4 (VBUS), J3.A9 (VBUS), J3.B4 (VBUS), J3.B9 (VBUS), L6.1, R23.2, U10.5 (VP), U9.4 (EN), U9.5 (VCC)
- new net +8V: C58.2, L8.2
- new net -8V: C57.2, L7.2
- new net D+: J3.A6 (D+), J3.B6 (D+), U10.1 (IO1), U12.7 (DP)
- new net D-: J3.A7 (D-), J3.B7 (D-), U10.3 (IO2), U12.8 (DM)
- new net IMAGE_MISO_{1}: R27.1
- new net IMAGE_MISO_{2}: R26.1
- new net IMAGE_MISO_{3}: R29.1
- new net IMAGE_MISO_{4}: R28.1
- no-connect marks 0 -> 7
Other:
- added sheet Sensor board 2 (sensor_board.kicad_sch)
- added sheet Sensor board 3 (sensor_board.kicad_sch)
- added sheet Sensor board 4 (sensor_board.kicad_sch)
- moved on the sheet: C75, C76, C77, C78, C79, C80, C81, C82, C83, C84, C85, C86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

Commit message: Fix shifted FMC D30 and D31 on main STM32
Pins for D30 and D31 were shifted up by one pin
Parts:
- added C?: 100nF, Capacitor_SMD:C_0402_1005Metric, symbol Device:C_Small
Connections:
- net +3V3: now also U11.9 (VDDQ), C?.1
- net FMC_D30: now also U14.11 (PI9); no longer U14.7 (PI8)
- net FMC_D31: now also U14.12 (PI10); no longer U14.11 (PI9)
- net GND: now also C?.2; no longer U11.9 (VSSQ)
- net IRQ_{3}: now also U14.7 (PI8); no longer U14.12 (PI10)
- net FMC_SDCKE1: no longer names the net of U14.84 (PH7)
Other:
- note removed: "TODO: - Check SDRAM pinout against datasheet"

Commit message: Use FC1-15-02-T-WT connector for RadEye1 modules
Parts:
- added H1, H2, H3, H4, H5: MH, MountingHole:MountingHole_3.2mm_M3_Pad_Via, symbol Mechanical:MountingHole_Pad
- gave numbers to parts that had none: 1
Connections:
- net GND: now also H1.1, H2.1, H3.1, H4.1, H5.1
