File: bioptics-bx4x4-dc44-camera-board.kicad_pcb (KiCad board)
At the start: 4 copper layers, 260 x 188 mm, 471 parts, among them J12 TagConnect_TC2030_SWD, J3 USB_C_Receptacle_USB2.0, J4 TagConnect_TC2030_SWD, J5 TagConnect_TC2030_SWD, J6 TagConnect_TC2030_SWD, J9 TagConnect_TC2030_SWD, U1 AMS1117-3.3, U10 SRV05-4, U11 IS4xS32160F-xTL, U12 USB3300-EZK, U13 AMS1117-3.3, U14 STM32H753IITx, U15 CJ431, U16 7408, U17 CJ431, U18 AMS1117-3.3, U19 STM32H753IITx, U2 STM32H753IITx, U20 7408, U21 SN74AVC8T245PW, U22 AD5112, U23 INA849, U24 SN74AVC8T245PW, U25 AD5112, U26 INA849, U27 CJ431, U28 AMS1117-3.3, U29 STM32H753IITx, U3 SN74AVC8T245PW, U30 7408, U31 SN74AVC8T245PW, U32 AD5112, U33 INA849, U34 SN74AVC8T245PW, U35 AD5112, U36 INA849, U37 CJ431, U38 AMS1117-3.3, U39 STM32H753IITx, U4 AD5112, U40 7408, U41 SN74AVC8T245PW, U42 AD5112, U43 INA849, U44 SN74AVC8T245PW, U45 AD5112, U46 INA849, U5 INA849, U6 SN74AVC8T245PW, U7 AD5112, U8 INA849, U9 FP6291, Y1 24MHz

Commit message: Use FC1-15-02-T-WT connector for RadEye1 modules
Parts:
- added C233: 100nF, Capacitor_SMD:C_0402_1005Metric, F.Cu at (357.4, 59.4)
- added H1: MH, MountingHole:MountingHole_3.2mm_M3_Pad_Via, F.Cu at (255.0, 206.3)
- added H2: MH, MountingHole:MountingHole_3.2mm_M3_Pad_Via, F.Cu at (256.5, 29.1)
- added H3: MH, MountingHole:MountingHole_3.2mm_M3_Pad_Via, F.Cu at (153.0, 134.0)
- added H4: MH, MountingHole:MountingHole_3.2mm_M3_Pad_Via, F.Cu at (52.0, 206.3)
- added H5: MH, MountingHole:MountingHole_3.2mm_M3_Pad_Via, F.Cu at (52.0, 29.1)
- added J1: RadEye1, Connector_Samtec_FC1:FC1-15-02-T-WT_P1.0mm, F.Cu at (426.0, -37.5)
- added J10: RadEye1, Connector_Samtec_FC1:FC1-15-02-T-WT_P1.0mm, F.Cu at (279.9, 37.8)
- added J11: RadEye1, Connector_Samtec_FC1:FC1-15-02-T-WT_P1.0mm, F.Cu at (399.8, -50.4)
- added J13: RadEye1, Connector_Samtec_FC1:FC1-15-02-T-WT_P1.0mm, F.Cu at (426.0, -50.4)
- added J14: RadEye1, Connector_Samtec_FC1:FC1-15-02-T-WT_P1.0mm, F.Cu at (452.2, -63.4)
- added J2: RadEye1, Connector_Samtec_FC1:FC1-15-02-T-WT_P1.0mm, F.Cu at (452.2, -50.4)
- added J7: RadEye1, Connector_Samtec_FC1:FC1-15-02-T-WT_P1.0mm, F.Cu at (426.0, -63.4)
- added J8: RadEye1, Connector_Samtec_FC1:FC1-15-02-T-WT_P1.0mm, F.Cu at (399.8, -37.5)
- moved U14 277.5 mm to (121.0, 173.0)
- moved U11 207.8 mm to (162.5, 174.0), turned to 180 degrees
- moved J3 173.7 mm to (27.9, 190.5)
- moved C232 170.3 mm to (38.3, 185.0)
- moved U10 170.3 mm to (35.8, 185.5)
- moved U12 170.3 mm to (43.0, 184.0)
- moved U29 84.7 mm to (356.0, 204.0)
Connections:
- U11 pad 9: GND -> +3V3
- U14 pad 11: /FMC_D31 -> /FMC_D30
- U14 pad 12: /IRQ_{3} -> /FMC_D31
- U14 pad 7: /FMC_D30 -> /IRQ_{3}
- U14 pad 84: /FMC_SDCKE1 -> unconnected-(U14-Pad84)
Other:
- board size 260 x 188 mm -> 260 x 187 mm

Commit message: First acquisition channel layout WiP
Parts:
- added C234: 100nF, Capacitor_SMD:C_0402_1005Metric, B.Cu at (62.9, 51.4)
- added C235: 100nF, Capacitor_SMD:C_0402_1005Metric, B.Cu at (341.3, 44.4)
- added C236: 100nF, Capacitor_SMD:C_0402_1005Metric, F.Cu at (345.7, 37.0)
- added C237: 100nF, Capacitor_SMD:C_0402_1005Metric, F.Cu at (352.5, 37.0)
- C10, C11, C12, C13, C14, C15, C16, C17, C18, C19, C20, C21, C22, C23, C24, C25, C26, C27, C30, C31, C32, C4, C5, C6, C7, C8, C9, FB2, FB3, FB4, L2, L3, R1, R2, R3, R37, R38, R39, R4, R5, R8, U16, U2, U3, U5, U6: moved to B.Cu
- moved FB2 518.1 mm to (38.8, 30.7)
- moved C5 517.5 mm to (62.5, 53.7), turned to 180 degrees
- moved C20 514.6 mm to (62.9, 57.6), turned to -90 degrees
- moved C27 508.0 mm to (36.4, 35.2), turned to -90 degrees
- moved C25 507.5 mm to (36.4, 31.2), turned to -90 degrees
- moved C7 506.2 mm to (61.9, 49.5), turned to -90 degrees
- moved C18 505.5 mm to (62.9, 49.5), turned to -90 degrees
- moved R4 505.4 mm to (36.8, 42.7)
- moved R5 505.3 mm to (36.8, 43.7)
- moved R1 503.9 mm to (62.5, 52.8)
- moved C4 503.8 mm to (75.0, 43.4), turned to 180 degrees
- moved C22 503.8 mm to (62.9, 61.6), turned to -90 degrees
- moved C24 502.2 mm to (43.1, 47.8)
- moved C21 501.2 mm to (67.7, 71.8), turned to 180 degrees
- moved R3 499.5 mm to (42.0, 33.6), turned to 180 degrees
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Connections:
- U21 pad 10: unconnected-(U21-Pad10) -> /Sensor board 2/Sensor 1/RESET_{5V}
- U21 pad 14: GND -> /Sensor board 2/RESET_{1}
- U21 pad 15: GND -> /Sensor board 2/START_{1}
- U21 pad 16: /Sensor board 2/ADC1_TRIG_OUT -> /Sensor board 2/CLOCK_{1}
- U21 pad 17: /Sensor board 2/NDR_{1} -> /Sensor board 2/BIN_{1}
- U21 pad 18: /Sensor board 2/BIN_{1} -> /Sensor board 2/NDR_{1}
- U21 pad 19: /Sensor board 2/CLOCK_{1} -> /Sensor board 2/ADC1_TRIG_OUT
- U21 pad 20: /Sensor board 2/START_{1} -> GND
- U21 pad 21: /Sensor board 2/RESET_{1} -> GND
- U21 pad 3: /Sensor board 2/Sensor 1/RESET_{5V} -> unconnected-(U21-Pad3)
- U21 pad 4: /Sensor board 2/Sensor 1/START_{5V} -> unconnected-(U21-Pad4)
- U21 pad 5: /Sensor board 2/Sensor 1/CLOCK_{5V} -> /Sensor board 2/Sensor 1/TRIG_OUT_{5V}
- U21 pad 6: /Sensor board 2/Sensor 1/BIN_{5V} -> /Sensor board 2/Sensor 1/NDR_{5V}
- U21 pad 7: /Sensor board 2/Sensor 1/NDR_{5V} -> /Sensor board 2/Sensor 1/BIN_{5V}
- U21 pad 8: /Sensor board 2/Sensor 1/TRIG_OUT_{5V} -> /Sensor board 2/Sensor 1/CLOCK_{5V}
- U21 pad 9: unconnected-(U21-Pad9) -> /Sensor board 2/Sensor 1/START_{5V}
- U23 pad 2: Net-(U22-Pad3) -> Net-(U22-Pad2)
- U23 pad 3: Net-(U22-Pad2) -> Net-(U22-Pad3)
- U24 pad 10: unconnected-(U24-Pad10) -> /Sensor board 2/Sensor 2/RESET_{5V}
- U24 pad 14: GND -> /Sensor board 2/RESET_{2}
- U24 pad 15: GND -> /Sensor board 2/START_{2}
- U24 pad 16: /Sensor board 2/ADC3_TRIG_OUT -> /Sensor board 2/CLOCK_{2}
- U24 pad 17: /Sensor board 2/NDR_{2} -> /Sensor board 2/BIN_{2}
- U24 pad 18: /Sensor board 2/BIN_{2} -> /Sensor board 2/NDR_{2}
- U24 pad 19: /Sensor board 2/CLOCK_{2} -> /Sensor board 2/ADC3_TRIG_OUT
- U24 pad 20: /Sensor board 2/START_{2} -> GND
- U24 pad 21: /Sensor board 2/RESET_{2} -> GND
- U24 pad 3: /Sensor board 2/Sensor 2/RESET_{5V} -> unconnected-(U24-Pad3)
- U24 pad 4: /Sensor board 2/Sensor 2/START_{5V} -> unconnected-(U24-Pad4)
- U24 pad 5: /Sensor board 2/Sensor 2/CLOCK_{5V} -> /Sensor board 2/Sensor 2/TRIG_OUT_{5V}
- U24 pad 6: /Sensor board 2/Sensor 2/BIN_{5V} -> /Sensor board 2/Sensor 2/NDR_{5V}
- U24 pad 7: /Sensor board 2/Sensor 2/NDR_{5V} -> /Sensor board 2/Sensor 2/BIN_{5V}
- U24 pad 8: /Sensor board 2/Sensor 2/TRIG_OUT_{5V} -> /Sensor board 2/Sensor 2/CLOCK_{5V}
- U24 pad 9: unconnected-(U24-Pad9) -> /Sensor board 2/Sensor 2/START_{5V}
- U26 pad 2: Net-(U25-Pad3) -> Net-(U25-Pad2)
- U26 pad 3: Net-(U25-Pad2) -> Net-(U25-Pad3)
- U3 pad 10: unconnected-(U3-Pad10) -> /Sensor board 1/Sensor 1/RESET_{5V}
- U3 pad 14: GND -> /Sensor board 1/RESET_{1}
- U3 pad 15: GND -> /Sensor board 1/START_{1}
- U3 pad 16: /Sensor board 1/ADC1_TRIG_OUT -> /Sensor board 1/CLOCK_{1}
- U3 pad 17: /Sensor board 1/NDR_{1} -> /Sensor board 1/BIN_{1}
- U3 pad 18: /Sensor board 1/BIN_{1} -> /Sensor board 1/NDR_{1}
- U3 pad 19: /Sensor board 1/CLOCK_{1} -> /Sensor board 1/ADC1_TRIG_OUT
- U3 pad 20: /Sensor board 1/START_{1} -> GND
- U3 pad 21: /Sensor board 1/RESET_{1} -> GND
- U3 pad 3: /Sensor board 1/Sensor 1/RESET_{5V} -> unconnected-(U3-Pad3)
- U3 pad 4: /Sensor board 1/Sensor 1/START_{5V} -> unconnected-(U3-Pad4)
- U3 pad 5: /Sensor board 1/Sensor 1/CLOCK_{5V} -> /Sensor board 1/Sensor 1/TRIG_OUT_{5V}
- U3 pad 6: /Sensor board 1/Sensor 1/BIN_{5V} -> /Sensor board 1/Sensor 1/NDR_{5V}
- U3 pad 7: /Sensor board 1/Sensor 1/NDR_{5V} -> /Sensor board 1/Sensor 1/BIN_{5V}
- U3 pad 8: /Sensor board 1/Sensor 1/TRIG_OUT_{5V} -> /Sensor board 1/Sensor 1/CLOCK_{5V}
- U3 pad 9: unconnected-(U3-Pad9) -> /Sensor board 1/Sensor 1/START_{5V}
- U31 pad 10: unconnected-(U31-Pad10) -> /Sensor board 3/Sensor 1/RESET_{5V}
- U31 pad 14: GND -> /Sensor board 3/RESET_{1}
- U31 pad 15: GND -> /Sensor board 3/START_{1}
- U31 pad 16: /Sensor board 3/ADC1_TRIG_OUT -> /Sensor board 3/CLOCK_{1}
- U31 pad 17: /Sensor board 3/NDR_{1} -> /Sensor board 3/BIN_{1}
- U31 pad 18: /Sensor board 3/BIN_{1} -> /Sensor board 3/NDR_{1}
- U31 pad 19: /Sensor board 3/CLOCK_{1} -> /Sensor board 3/ADC1_TRIG_OUT
- U31 pad 20: /Sensor board 3/START_{1} -> GND
- U31 pad 21: /Sensor board 3/RESET_{1} -> GND
- U31 pad 3: /Sensor board 3/Sensor 1/RESET_{5V} -> unconnected-(U31-Pad3)
- U31 pad 4: /Sensor board 3/Sensor 1/START_{5V} -> unconnected-(U31-Pad4)
- U31 pad 5: /Sensor board 3/Sensor 1/CLOCK_{5V} -> /Sensor board 3/Sensor 1/TRIG_OUT_{5V}
- U31 pad 6: /Sensor board 3/Sensor 1/BIN_{5V} -> /Sensor board 3/Sensor 1/NDR_{5V}
- U31 pad 7: /Sensor board 3/Sensor 1/NDR_{5V} -> /Sensor board 3/Sensor 1/BIN_{5V}
- U31 pad 8: /Sensor board 3/Sensor 1/TRIG_OUT_{5V} -> /Sensor board 3/Sensor 1/CLOCK_{5V}
- U31 pad 9: unconnected-(U31-Pad9) -> /Sensor board 3/Sensor 1/START_{5V}
- U33 pad 2: Net-(U32-Pad3) -> Net-(U32-Pad2)
- U33 pad 3: Net-(U32-Pad2) -> Net-(U32-Pad3)
- U34 pad 10: unconnected-(U34-Pad10) -> /Sensor board 3/Sensor 2/RESET_{5V}
- U34 pad 14: GND -> /Sensor board 3/RESET_{2}
- U34 pad 15: GND -> /Sensor board 3/START_{2}
- U34 pad 16: /Sensor board 3/ADC3_TRIG_OUT -> /Sensor board 3/CLOCK_{2}
- U34 pad 17: /Sensor board 3/NDR_{2} -> /Sensor board 3/BIN_{2}
- U34 pad 18: /Sensor board 3/BIN_{2} -> /Sensor board 3/NDR_{2}
- U34 pad 19: /Sensor board 3/CLOCK_{2} -> /Sensor board 3/ADC3_TRIG_OUT
- U34 pad 20: /Sensor board 3/START_{2} -> GND
- U34 pad 21: /Sensor board 3/RESET_{2} -> GND
- U34 pad 3: /Sensor board 3/Sensor 2/RESET_{5V} -> unconnected-(U34-Pad3)
- U34 pad 4: /Sensor board 3/Sensor 2/START_{5V} -> unconnected-(U34-Pad4)
- U34 pad 5: /Sensor board 3/Sensor 2/CLOCK_{5V} -> /Sensor board 3/Sensor 2/TRIG_OUT_{5V}
- U34 pad 6: /Sensor board 3/Sensor 2/BIN_{5V} -> /Sensor board 3/Sensor 2/NDR_{5V}
- U34 pad 7: /Sensor board 3/Sensor 2/NDR_{5V} -> /Sensor board 3/Sensor 2/BIN_{5V}
- U34 pad 8: /Sensor board 3/Sensor 2/TRIG_OUT_{5V} -> /Sensor board 3/Sensor 2/CLOCK_{5V}
- U34 pad 9: unconnected-(U34-Pad9) -> /Sensor board 3/Sensor 2/START_{5V}
- U36 pad 2: Net-(U35-Pad3) -> Net-(U35-Pad2)
- U36 pad 3: Net-(U35-Pad2) -> Net-(U35-Pad3)
- U41 pad 10: unconnected-(U41-Pad10) -> /Sensor board 4/Sensor 1/RESET_{5V}
- U41 pad 14: GND -> /Sensor board 4/RESET_{1}
- U41 pad 15: GND -> /Sensor board 4/START_{1}
- U41 pad 16: /Sensor board 4/ADC1_TRIG_OUT -> /Sensor board 4/CLOCK_{1}
- U41 pad 17: /Sensor board 4/NDR_{1} -> /Sensor board 4/BIN_{1}
- U41 pad 18: /Sensor board 4/BIN_{1} -> /Sensor board 4/NDR_{1}
- U41 pad 19: /Sensor board 4/CLOCK_{1} -> /Sensor board 4/ADC1_TRIG_OUT
- U41 pad 20: /Sensor board 4/START_{1} -> GND
- U41 pad 21: /Sensor board 4/RESET_{1} -> GND
- U41 pad 3: /Sensor board 4/Sensor 1/RESET_{5V} -> unconnected-(U41-Pad3)
- U41 pad 4: /Sensor board 4/Sensor 1/START_{5V} -> unconnected-(U41-Pad4)
- U41 pad 5: /Sensor board 4/Sensor 1/CLOCK_{5V} -> /Sensor board 4/Sensor 1/TRIG_OUT_{5V}
- U41 pad 6: /Sensor board 4/Sensor 1/BIN_{5V} -> /Sensor board 4/Sensor 1/NDR_{5V}
- U41 pad 7: /Sensor board 4/Sensor 1/NDR_{5V} -> /Sensor board 4/Sensor 1/BIN_{5V}
- U41 pad 8: /Sensor board 4/Sensor 1/TRIG_OUT_{5V} -> /Sensor board 4/Sensor 1/CLOCK_{5V}
- U41 pad 9: unconnected-(U41-Pad9) -> /Sensor board 4/Sensor 1/START_{5V}
- U43 pad 2: Net-(U42-Pad3) -> Net-(U42-Pad2)
- U43 pad 3: Net-(U42-Pad2) -> Net-(U42-Pad3)
- U44 pad 10: unconnected-(U44-Pad10) -> /Sensor board 4/Sensor 2/RESET_{5V}
- U44 pad 14: GND -> /Sensor board 4/RESET_{2}
- U44 pad 15: GND -> /Sensor board 4/START_{2}
- U44 pad 16: /Sensor board 4/ADC3_TRIG_OUT -> /Sensor board 4/CLOCK_{2}
- U44 pad 17: /Sensor board 4/NDR_{2} -> /Sensor board 4/BIN_{2}
- U44 pad 18: /Sensor board 4/BIN_{2} -> /Sensor board 4/NDR_{2}
- U44 pad 19: /Sensor board 4/CLOCK_{2} -> /Sensor board 4/ADC3_TRIG_OUT
- U44 pad 20: /Sensor board 4/START_{2} -> GND
- U44 pad 21: /Sensor board 4/RESET_{2} -> GND
- U44 pad 3: /Sensor board 4/Sensor 2/RESET_{5V} -> unconnected-(U44-Pad3)
- U44 pad 4: /Sensor board 4/Sensor 2/START_{5V} -> unconnected-(U44-Pad4)
- U44 pad 5: /Sensor board 4/Sensor 2/CLOCK_{5V} -> /Sensor board 4/Sensor 2/TRIG_OUT_{5V}
- U44 pad 6: /Sensor board 4/Sensor 2/BIN_{5V} -> /Sensor board 4/Sensor 2/NDR_{5V}
- U44 pad 7: /Sensor board 4/Sensor 2/NDR_{5V} -> /Sensor board 4/Sensor 2/BIN_{5V}
- U44 pad 8: /Sensor board 4/Sensor 2/TRIG_OUT_{5V} -> /Sensor board 4/Sensor 2/CLOCK_{5V}
- U44 pad 9: unconnected-(U44-Pad9) -> /Sensor board 4/Sensor 2/START_{5V}
- U46 pad 2: Net-(U45-Pad3) -> Net-(U45-Pad2)
- U46 pad 3: Net-(U45-Pad2) -> Net-(U45-Pad3)
- U5 pad 2: Net-(U4-Pad3) -> Net-(U4-Pad2)
- U5 pad 3: Net-(U4-Pad2) -> Net-(U4-Pad3)
- U6 pad 10: unconnected-(U6-Pad10) -> /Sensor board 1/Sensor 2/RESET_{5V}
- U6 pad 14: GND -> /Sensor board 1/RESET_{2}
- U6 pad 15: GND -> /Sensor board 1/START_{2}
- U6 pad 16: /Sensor board 1/ADC3_TRIG_OUT -> /Sensor board 1/CLOCK_{2}
- U6 pad 17: /Sensor board 1/NDR_{2} -> /Sensor board 1/BIN_{2}
- U6 pad 18: /Sensor board 1/BIN_{2} -> /Sensor board 1/NDR_{2}
- U6 pad 19: /Sensor board 1/CLOCK_{2} -> /Sensor board 1/ADC3_TRIG_OUT
- U6 pad 20: /Sensor board 1/START_{2} -> GND
- U6 pad 21: /Sensor board 1/RESET_{2} -> GND
- U6 pad 3: /Sensor board 1/Sensor 2/RESET_{5V} -> unconnected-(U6-Pad3)
- U6 pad 4: /Sensor board 1/Sensor 2/START_{5V} -> unconnected-(U6-Pad4)
- U6 pad 5: /Sensor board 1/Sensor 2/CLOCK_{5V} -> /Sensor board 1/Sensor 2/TRIG_OUT_{5V}
- U6 pad 6: /Sensor board 1/Sensor 2/BIN_{5V} -> /Sensor board 1/Sensor 2/NDR_{5V}
- U6 pad 7: /Sensor board 1/Sensor 2/NDR_{5V} -> /Sensor board 1/Sensor 2/BIN_{5V}
- U6 pad 8: /Sensor board 1/Sensor 2/TRIG_OUT_{5V} -> /Sensor board 1/Sensor 2/CLOCK_{5V}
- U6 pad 9: unconnected-(U6-Pad9) -> /Sensor board 1/Sensor 2/START_{5V}
- U8 pad 2: Net-(U7-Pad3) -> Net-(U7-Pad2)
- U8 pad 3: Net-(U7-Pad2) -> Net-(U7-Pad3)
Routing:
- net GND: track 1.68 -> 79.7 mm, vias 0 -> 34
- net /Sensor board 1/3v3: track 0.00 -> 41.6 mm, vias 0 -> 16
- net /Sensor board 1/Sensor 1/S+: track 0.00 -> 20.9 mm
- net /Sensor board 1/Sensor 1/S-: track 0.00 -> 20.4 mm
- net Net-(R8-Pad1): track 0.00 -> 9.58 mm
- net /Sensor board 1/Sensor 1/RESET_{5V}: track 0.00 -> 9.51 mm, vias 0 -> 1
- net /Sensor board 1/Sensor 1/START_{5V}: track 0.00 -> 9.28 mm, vias 0 -> 1
- net /Sensor board 1/Sensor 1/CLOCK_{5V}: track 0.00 -> 9.22 mm, vias 0 -> 1
- net /Sensor board 1/Sensor 1/BIN_{5V}: track 0.00 -> 8.99 mm, vias 0 -> 1
- net /Sensor board 1/Sensor 1/NDR_{5V}: track 0.00 -> 8.87 mm, vias 0 -> 1
- net Net-(J1-Pad4): track 0.00 -> 7.29 mm, vias 0 -> 1
- net Net-(J1-Pad3): track 0.00 -> 7.26 mm, vias 0 -> 1
- net Net-(C29-Pad1): track 0.00 -> 6.45 mm, vias 0 -> 1
- net /Sensor board 1/3v3A: track 0.00 -> 4.43 mm
- net Net-(C30-Pad2): track 0.00 -> 4.38 mm
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
Commit message: Layout first sensor pair
Parts:
- added D4: 1N4148WS, Diode_SMD:D_SOD-323, F.Cu at (349.6, -12.4)
- added D5: 1N4148WS, Diode_SMD:D_SOD-323, F.Cu at (133.9, 33.1)
- added D6: 1N4148WS, Diode_SMD:D_SOD-323, F.Cu at (340.9, -18.6)
- added D7: 1N4148WS, Diode_SMD:D_SOD-323, F.Cu at (349.6, -18.6)
- C10, C11, C12, C13, C14, C15, C16, C17, C18, C19, C20, C21, C22, C23, C234, C24, C25, C26, C27, C30, C31, C32, C4, C5, C6, C7, C8, C9, FB2, FB3, FB4, L2, L3, R1, R2, R3, R37, R38, R39, R4, R5, R8, U16, U2, U3, U5, U6: moved to F.Cu
- moved C37 570.8 mm to (33.5, 59.8), turned to -90 degrees
- moved C35 569.7 mm to (33.5, 55.8), turned to -90 degrees
- moved R11 560.8 mm to (42.3, 64.7), turned to 45 degrees
- moved R12 559.9 mm to (43.0, 65.4), turned to 45 degrees
- moved L4 559.7 mm to (33.1, 62.6), turned to -90 degrees
- moved C34 557.6 mm to (46.8, 57.3)
- moved R10 554.7 mm to (45.8, 51.1), turned to 180 degrees
- moved R9 554.2 mm to (45.8, 52.0)
- moved C33 548.8 mm to (51.6, 57.3)
- moved U6 547.6 mm to (49.2, 62.0), turned to 0 degrees
- moved C38 546.1 mm to (60.5, 49.0), turned to 180 degrees
- moved C36 546.1 mm to (47.2, 51.6), turned to -90 degrees
- moved U7 546.0 mm to (60.5, 51.6), turned to 90 degrees
- moved C40 542.1 mm to (65.1, 55.1), turned to 90 degrees
- moved L5 538.4 mm to (63.9, 50.4)
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Connections:
- U19 pad 35: /Sensor board 2/sensor2_out -> /Sensor board 2/sensor1_out
- U19 pad 59: /Sensor board 2/sensor1_out -> /Sensor board 2/sensor2_out
- U2 pad 35: /Sensor board 1/sensor2_out -> /Sensor board 1/sensor1_out
- U2 pad 59: /Sensor board 1/sensor1_out -> /Sensor board 1/sensor2_out
- U21 pad 10: /Sensor board 2/Sensor 1/RESET_{5V} -> unconnected-(U21-Pad10)
- U21 pad 14: /Sensor board 2/RESET_{1} -> GND
- U21 pad 15: /Sensor board 2/START_{1} -> GND
- U21 pad 16: /Sensor board 2/CLOCK_{1} -> /Sensor board 2/ADC1_TRIG_OUT
- U21 pad 17: /Sensor board 2/BIN_{1} -> /Sensor board 2/NDR_{1}
- U21 pad 18: /Sensor board 2/NDR_{1} -> /Sensor board 2/BIN_{1}
- U21 pad 19: /Sensor board 2/ADC1_TRIG_OUT -> /Sensor board 2/CLOCK_{1}
- U21 pad 20: GND -> /Sensor board 2/START_{1}
- U21 pad 21: GND -> /Sensor board 2/RESET_{1}
- U21 pad 3: unconnected-(U21-Pad3) -> /Sensor board 2/Sensor 1/RESET_{5V}
- U21 pad 4: unconnected-(U21-Pad4) -> /Sensor board 2/Sensor 1/START_{5V}
- U21 pad 5: /Sensor board 2/Sensor 1/TRIG_OUT_{5V} -> /Sensor board 2/Sensor 1/CLOCK_{5V}
- U21 pad 6: /Sensor board 2/Sensor 1/NDR_{5V} -> /Sensor board 2/Sensor 1/BIN_{5V}
- U21 pad 7: /Sensor board 2/Sensor 1/BIN_{5V} -> /Sensor board 2/Sensor 1/NDR_{5V}
- U21 pad 8: /Sensor board 2/Sensor 1/CLOCK_{5V} -> /Sensor board 2/Sensor 1/TRIG_OUT_{5V}
- U21 pad 9: /Sensor board 2/Sensor 1/START_{5V} -> unconnected-(U21-Pad9)
- U24 pad 10: /Sensor board 2/Sensor 2/RESET_{5V} -> unconnected-(U24-Pad10)
- U24 pad 14: /Sensor board 2/RESET_{2} -> GND
- U24 pad 15: /Sensor board 2/START_{2} -> GND
- U24 pad 16: /Sensor board 2/CLOCK_{2} -> /Sensor board 2/ADC3_TRIG_OUT
- U24 pad 17: /Sensor board 2/BIN_{2} -> /Sensor board 2/NDR_{2}
- U24 pad 18: /Sensor board 2/NDR_{2} -> /Sensor board 2/BIN_{2}
- U24 pad 19: /Sensor board 2/ADC3_TRIG_OUT -> /Sensor board 2/CLOCK_{2}
- U24 pad 20: GND -> /Sensor board 2/START_{2}
- U24 pad 21: GND -> /Sensor board 2/RESET_{2}
- U24 pad 3: unconnected-(U24-Pad3) -> /Sensor board 2/Sensor 2/RESET_{5V}
- U24 pad 4: unconnected-(U24-Pad4) -> /Sensor board 2/Sensor 2/START_{5V}
- U24 pad 5: /Sensor board 2/Sensor 2/TRIG_OUT_{5V} -> /Sensor board 2/Sensor 2/CLOCK_{5V}
- U24 pad 6: /Sensor board 2/Sensor 2/NDR_{5V} -> /Sensor board 2/Sensor 2/BIN_{5V}
- U24 pad 7: /Sensor board 2/Sensor 2/BIN_{5V} -> /Sensor board 2/Sensor 2/NDR_{5V}
- U24 pad 8: /Sensor board 2/Sensor 2/CLOCK_{5V} -> /Sensor board 2/Sensor 2/TRIG_OUT_{5V}
- U24 pad 9: /Sensor board 2/Sensor 2/START_{5V} -> unconnected-(U24-Pad9)
- U29 pad 35: /Sensor board 3/sensor2_out -> /Sensor board 3/sensor1_out
- U29 pad 59: /Sensor board 3/sensor1_out -> /Sensor board 3/sensor2_out
- U3 pad 10: /Sensor board 1/Sensor 1/RESET_{5V} -> unconnected-(U3-Pad10)
- U3 pad 14: /Sensor board 1/RESET_{1} -> GND
- U3 pad 15: /Sensor board 1/START_{1} -> GND
- U3 pad 16: /Sensor board 1/CLOCK_{1} -> /Sensor board 1/ADC1_TRIG_OUT
- U3 pad 17: /Sensor board 1/BIN_{1} -> /Sensor board 1/NDR_{1}
- U3 pad 18: /Sensor board 1/NDR_{1} -> /Sensor board 1/BIN_{1}
- U3 pad 19: /Sensor board 1/ADC1_TRIG_OUT -> /Sensor board 1/CLOCK_{1}
- U3 pad 20: GND -> /Sensor board 1/START_{1}
- U3 pad 21: GND -> /Sensor board 1/RESET_{1}
- U3 pad 3: unconnected-(U3-Pad3) -> /Sensor board 1/Sensor 1/RESET_{5V}
- U3 pad 4: unconnected-(U3-Pad4) -> /Sensor board 1/Sensor 1/START_{5V}
- U3 pad 5: /Sensor board 1/Sensor 1/TRIG_OUT_{5V} -> /Sensor board 1/Sensor 1/CLOCK_{5V}
- U3 pad 6: /Sensor board 1/Sensor 1/NDR_{5V} -> /Sensor board 1/Sensor 1/BIN_{5V}
- U3 pad 7: /Sensor board 1/Sensor 1/BIN_{5V} -> /Sensor board 1/Sensor 1/NDR_{5V}
- U3 pad 8: /Sensor board 1/Sensor 1/CLOCK_{5V} -> /Sensor board 1/Sensor 1/TRIG_OUT_{5V}
- U3 pad 9: /Sensor board 1/Sensor 1/START_{5V} -> unconnected-(U3-Pad9)
- U31 pad 10: /Sensor board 3/Sensor 1/RESET_{5V} -> unconnected-(U31-Pad10)
- U31 pad 14: /Sensor board 3/RESET_{1} -> GND
- U31 pad 15: /Sensor board 3/START_{1} -> GND
- U31 pad 16: /Sensor board 3/CLOCK_{1} -> /Sensor board 3/ADC1_TRIG_OUT
- U31 pad 17: /Sensor board 3/BIN_{1} -> /Sensor board 3/NDR_{1}
- U31 pad 18: /Sensor board 3/NDR_{1} -> /Sensor board 3/BIN_{1}
- U31 pad 19: /Sensor board 3/ADC1_TRIG_OUT -> /Sensor board 3/CLOCK_{1}
- U31 pad 20: GND -> /Sensor board 3/START_{1}
- U31 pad 21: GND -> /Sensor board 3/RESET_{1}
- U31 pad 3: unconnected-(U31-Pad3) -> /Sensor board 3/Sensor 1/RESET_{5V}
- U31 pad 4: unconnected-(U31-Pad4) -> /Sensor board 3/Sensor 1/START_{5V}
- U31 pad 5: /Sensor board 3/Sensor 1/TRIG_OUT_{5V} -> /Sensor board 3/Sensor 1/CLOCK_{5V}
- U31 pad 6: /Sensor board 3/Sensor 1/NDR_{5V} -> /Sensor board 3/Sensor 1/BIN_{5V}
- U31 pad 7: /Sensor board 3/Sensor 1/BIN_{5V} -> /Sensor board 3/Sensor 1/NDR_{5V}
- U31 pad 8: /Sensor board 3/Sensor 1/CLOCK_{5V} -> /Sensor board 3/Sensor 1/TRIG_OUT_{5V}
- U31 pad 9: /Sensor board 3/Sensor 1/START_{5V} -> unconnected-(U31-Pad9)
- U34 pad 10: /Sensor board 3/Sensor 2/RESET_{5V} -> unconnected-(U34-Pad10)
- U34 pad 14: /Sensor board 3/RESET_{2} -> GND
- U34 pad 15: /Sensor board 3/START_{2} -> GND
- U34 pad 16: /Sensor board 3/CLOCK_{2} -> /Sensor board 3/ADC3_TRIG_OUT
- U34 pad 17: /Sensor board 3/BIN_{2} -> /Sensor board 3/NDR_{2}
- U34 pad 18: /Sensor board 3/NDR_{2} -> /Sensor board 3/BIN_{2}
- U34 pad 19: /Sensor board 3/ADC3_TRIG_OUT -> /Sensor board 3/CLOCK_{2}
- U34 pad 20: GND -> /Sensor board 3/START_{2}
- U34 pad 21: GND -> /Sensor board 3/RESET_{2}
- U34 pad 3: unconnected-(U34-Pad3) -> /Sensor board 3/Sensor 2/RESET_{5V}
- U34 pad 4: unconnected-(U34-Pad4) -> /Sensor board 3/Sensor 2/START_{5V}
- U34 pad 5: /Sensor board 3/Sensor 2/TRIG_OUT_{5V} -> /Sensor board 3/Sensor 2/CLOCK_{5V}
- U34 pad 6: /Sensor board 3/Sensor 2/NDR_{5V} -> /Sensor board 3/Sensor 2/BIN_{5V}
- U34 pad 7: /Sensor board 3/Sensor 2/BIN_{5V} -> /Sensor board 3/Sensor 2/NDR_{5V}
- U34 pad 8: /Sensor board 3/Sensor 2/CLOCK_{5V} -> /Sensor board 3/Sensor 2/TRIG_OUT_{5V}
- U34 pad 9: /Sensor board 3/Sensor 2/START_{5V} -> unconnected-(U34-Pad9)
- U39 pad 35: /Sensor board 4/sensor2_out -> /Sensor board 4/sensor1_out
- U39 pad 59: /Sensor board 4/sensor1_out -> /Sensor board 4/sensor2_out
- U41 pad 10: /Sensor board 4/Sensor 1/RESET_{5V} -> unconnected-(U41-Pad10)
- U41 pad 14: /Sensor board 4/RESET_{1} -> GND
- U41 pad 15: /Sensor board 4/START_{1} -> GND
- U41 pad 16: /Sensor board 4/CLOCK_{1} -> /Sensor board 4/ADC1_TRIG_OUT
- U41 pad 17: /Sensor board 4/BIN_{1} -> /Sensor board 4/NDR_{1}
- U41 pad 18: /Sensor board 4/NDR_{1} -> /Sensor board 4/BIN_{1}
- U41 pad 19: /Sensor board 4/ADC1_TRIG_OUT -> /Sensor board 4/CLOCK_{1}
- U41 pad 20: GND -> /Sensor board 4/START_{1}
- U41 pad 21: GND -> /Sensor board 4/RESET_{1}
- U41 pad 3: unconnected-(U41-Pad3) -> /Sensor board 4/Sensor 1/RESET_{5V}
- U41 pad 4: unconnected-(U41-Pad4) -> /Sensor board 4/Sensor 1/START_{5V}
- U41 pad 5: /Sensor board 4/Sensor 1/TRIG_OUT_{5V} -> /Sensor board 4/Sensor 1/CLOCK_{5V}
- U41 pad 6: /Sensor board 4/Sensor 1/NDR_{5V} -> /Sensor board 4/Sensor 1/BIN_{5V}
- U41 pad 7: /Sensor board 4/Sensor 1/BIN_{5V} -> /Sensor board 4/Sensor 1/NDR_{5V}
- U41 pad 8: /Sensor board 4/Sensor 1/CLOCK_{5V} -> /Sensor board 4/Sensor 1/TRIG_OUT_{5V}
- U41 pad 9: /Sensor board 4/Sensor 1/START_{5V} -> unconnected-(U41-Pad9)
- U44 pad 10: /Sensor board 4/Sensor 2/RESET_{5V} -> unconnected-(U44-Pad10)
- U44 pad 14: /Sensor board 4/RESET_{2} -> GND
- U44 pad 15: /Sensor board 4/START_{2} -> GND
- U44 pad 16: /Sensor board 4/CLOCK_{2} -> /Sensor board 4/ADC3_TRIG_OUT
- U44 pad 17: /Sensor board 4/BIN_{2} -> /Sensor board 4/NDR_{2}
- U44 pad 18: /Sensor board 4/NDR_{2} -> /Sensor board 4/BIN_{2}
- U44 pad 19: /Sensor board 4/ADC3_TRIG_OUT -> /Sensor board 4/CLOCK_{2}
- U44 pad 20: GND -> /Sensor board 4/START_{2}
- U44 pad 21: GND -> /Sensor board 4/RESET_{2}
- U44 pad 3: unconnected-(U44-Pad3) -> /Sensor board 4/Sensor 2/RESET_{5V}
- U44 pad 4: unconnected-(U44-Pad4) -> /Sensor board 4/Sensor 2/START_{5V}
- U44 pad 5: /Sensor board 4/Sensor 2/TRIG_OUT_{5V} -> /Sensor board 4/Sensor 2/CLOCK_{5V}
- U44 pad 6: /Sensor board 4/Sensor 2/NDR_{5V} -> /Sensor board 4/Sensor 2/BIN_{5V}
- U44 pad 7: /Sensor board 4/Sensor 2/BIN_{5V} -> /Sensor board 4/Sensor 2/NDR_{5V}
- U44 pad 8: /Sensor board 4/Sensor 2/CLOCK_{5V} -> /Sensor board 4/Sensor 2/TRIG_OUT_{5V}
- U44 pad 9: /Sensor board 4/Sensor 2/START_{5V} -> unconnected-(U44-Pad9)
- U6 pad 10: /Sensor board 1/Sensor 2/RESET_{5V} -> unconnected-(U6-Pad10)
- U6 pad 14: /Sensor board 1/RESET_{2} -> GND
- U6 pad 15: /Sensor board 1/START_{2} -> GND
- U6 pad 16: /Sensor board 1/CLOCK_{2} -> /Sensor board 1/ADC3_TRIG_OUT
- U6 pad 17: /Sensor board 1/BIN_{2} -> /Sensor board 1/NDR_{2}
- U6 pad 18: /Sensor board 1/NDR_{2} -> /Sensor board 1/BIN_{2}
- U6 pad 19: /Sensor board 1/ADC3_TRIG_OUT -> /Sensor board 1/CLOCK_{2}
- U6 pad 20: GND -> /Sensor board 1/START_{2}
- U6 pad 21: GND -> /Sensor board 1/RESET_{2}
- U6 pad 3: unconnected-(U6-Pad3) -> /Sensor board 1/Sensor 2/RESET_{5V}
- U6 pad 4: unconnected-(U6-Pad4) -> /Sensor board 1/Sensor 2/START_{5V}
- U6 pad 5: /Sensor board 1/Sensor 2/TRIG_OUT_{5V} -> /Sensor board 1/Sensor 2/CLOCK_{5V}
- U6 pad 6: /Sensor board 1/Sensor 2/NDR_{5V} -> /Sensor board 1/Sensor 2/BIN_{5V}
- U6 pad 7: /Sensor board 1/Sensor 2/BIN_{5V} -> /Sensor board 1/Sensor 2/NDR_{5V}
- U6 pad 8: /Sensor board 1/Sensor 2/CLOCK_{5V} -> /Sensor board 1/Sensor 2/TRIG_OUT_{5V}
- U6 pad 9: /Sensor board 1/Sensor 2/START_{5V} -> unconnected-(U6-Pad9)
Routing:
- net GND: track 79.7 -> 187.5 mm, vias 34 -> 45
- net Net-(J5-Pad2): track 0.00 -> 101.0 mm, vias 0 -> 3
- net Net-(J5-Pad4): track 0.00 -> 99.5 mm, vias 0 -> 3
- net /Sensor board 1/JTDO: track 0.00 -> 97.2 mm, vias 0 -> 3
- net /SLAVE_~{RST}: track 1.47 -> 97.8 mm, vias 0 -> 4
- net /Sensor board 1/RESET_{1}: track 0.00 -> 81.1 mm, vias 0 -> 2
- net /Sensor board 1/START_{1}: track 0.00 -> 81.1 mm, vias 0 -> 2
- net /Sensor board 1/CLOCK_{1}: track 0.00 -> 80.7 mm, vias 0 -> 2
- net /Sensor board 1/NDR_{1}: track 0.00 -> 76.7 mm, vias 0 -> 2
- net /Sensor board 1/BIN_{1}: track 0.00 -> 76.0 mm, vias 0 -> 2
- net /Sensor board 1/LINE_{1}: track 0.00 -> 72.1 mm, vias 0 -> 4
- net /Sensor board 1/FRAME_{1}: track 0.00 -> 70.5 mm, vias 0 -> 4
- net /Sensor board 1/RESET_{2}: track 0.00 -> 53.1 mm, vias 0 -> 2
- net /Sensor board 1/START_{2}: track 0.00 -> 52.6 mm, vias 0 -> 2
- net /Sensor board 1/FRAME_{2}: track 0.00 -> 52.3 mm, vias 0 -> 3
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
Commit message: Center snsor MCU between sensor connectors
Parts:
- removed C143, C188: 1uF, Capacitor_SMD:C_0402_1005Metric
- removed C145, C190: 100nF, Capacitor_SMD:C_0402_1005Metric
- removed FB21, FB30: 600R@100MHz, Inductor_SMD:L_0805_2012Metric
- removed L17, L23: 10uH, Inductor_SMD:L_0805_2012Metric
- removed R64, R87: 5.1k, Resistor_SMD:R_0402_1005Metric
- removed R65, R88: 100, Resistor_SMD:R_0402_1005Metric
- removed R66, R89: 10k, Resistor_SMD:R_0402_1005Metric
- removed R67, R90: 120, Resistor_SMD:R_0805_2012Metric
- removed U27, U37: CJ431, Package_TO_SOT_SMD:SOT-23
- moved R13 493.1 mm to (56.6, 48.8), turned to -90 degrees
- moved R6 490.8 mm to (59.1, 28.7), turned to -90 degrees
- moved R14 474.8 mm to (57.5, 48.8), turned to -90 degrees
- moved R7 472.2 mm to (60.1, 28.7), turned to -90 degrees
- moved C3 465.4 mm to (104.3, 35.0), turned to 90 degrees
- moved C1 442.9 mm to (140.8, 50.2), turned to -90 degrees
- moved L1 432.7 mm to (102.0, 35.5)
- moved U1 425.0 mm to (146.3, 50.2)
- moved FB1 414.6 mm to (143.2, 55.7), turned to -90 degrees
- moved C2 398.3 mm to (144.3, 46.1), turned to 180 degrees
- moved C95 349.3 mm to (44.7, 69.6), turned to 90 degrees
- moved L10 342.2 mm to (45.8, 71.4), turned to 180 degrees
- moved R35 340.6 mm to (49.2, 68.2), turned to 180 degrees
- moved U15 338.0 mm to (49.6, 70.5), turned to 180 degrees
- moved R33 336.0 mm to (52.5, 69.3), turned to 90 degrees
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Connections:
- C100 pad 1: /Sensor board 2/3v8 -> /3v8_2
- C103 pad 1: /SLAVE_~{RST} -> /Sensor board 2/MCUL_~{RST}
- C148 pad 1: /SLAVE_~{RST} -> /Sensor board 3/MCUL_~{RST}
- C193 pad 1: /SLAVE_~{RST} -> /Sensor board 4/MCUL_~{RST}
- C5 pad 1: /SLAVE_~{RST} -> /Sensor board 1/MCUL_~{RST}
- C95 pad 1: /Sensor board 1/3v8 -> /3v8_1
- D4 pad 2: /SLAVE_~{RST} -> /Sensor board 1/MCUL_~{RST}
- D5 pad 2: /SLAVE_~{RST} -> /Sensor board 2/MCUL_~{RST}
- D6 pad 2: /SLAVE_~{RST} -> /Sensor board 3/MCUL_~{RST}
- D7 pad 2: /SLAVE_~{RST} -> /Sensor board 4/MCUL_~{RST}
- J12 pad 3: /SLAVE_~{RST} -> /Sensor board 4/MCUL_~{RST}
- J5 pad 3: /SLAVE_~{RST} -> /Sensor board 1/MCUL_~{RST}
- J6 pad 3: /SLAVE_~{RST} -> /Sensor board 2/MCUL_~{RST}
- J9 pad 3: /SLAVE_~{RST} -> /Sensor board 3/MCUL_~{RST}
- L10 pad 2: /Sensor board 1/3v8 -> /3v8_1
- L11 pad 2: /Sensor board 2/3v8 -> /3v8_2
- L13 pad 2: /Sensor board 2/3v8 -> /3v8_1
- L15 pad 2: /Sensor board 2/3v8 -> /3v8_1
- L19 pad 2: /Sensor board 3/3v8 -> /3v8_2
- L2 pad 2: /Sensor board 1/3v8 -> /3v8_1
- L21 pad 2: /Sensor board 3/3v8 -> /3v8_2
- L25 pad 2: /Sensor board 4/3v8 -> /3v8_2
- L27 pad 2: /Sensor board 4/3v8 -> /3v8_2
- L4 pad 2: /Sensor board 1/3v8 -> /3v8_1
- R1 pad 2: /SLAVE_~{RST} -> /Sensor board 1/MCUL_~{RST}
- R37 pad 2: /IMAGE_FRAME_{1} -> /IMAGE_~{FRAME}_{1}
- R45 pad 2: /SLAVE_~{RST} -> /Sensor board 2/MCUL_~{RST}
- R46 pad 2: /IMAGE_FRAME_{2} -> /IMAGE_~{FRAME}_{2}
- R68 pad 2: /SLAVE_~{RST} -> /Sensor board 3/MCUL_~{RST}
- R69 pad 2: /IMAGE_FRAME_{3} -> /IMAGE_~{FRAME}_{3}
- R91 pad 2: /SLAVE_~{RST} -> /Sensor board 4/MCUL_~{RST}
- R92 pad 2: /IMAGE_FRAME_{4} -> /IMAGE_~{FRAME}_{4}
- U14 pad 1: /IMAGE_SCK_{3} -> /IMAGE_CLK_{3}
- U14 pad 145: /IMAGE_SCK_{4} -> /IMAGE_CLK_{4}
- U14 pad 156: /IMAGE_SCK_{2} -> /IMAGE_CLK_{2}
- U14 pad 25: /IMAGE_SCK_{1} -> /IMAGE_CLK_{1}
- U19 pad 31: /SLAVE_~{RST} -> /Sensor board 2/MCUL_~{RST}
- U2 pad 31: /SLAVE_~{RST} -> /Sensor board 1/MCUL_~{RST}
- U29 pad 31: /SLAVE_~{RST} -> /Sensor board 3/MCUL_~{RST}
- U39 pad 31: /SLAVE_~{RST} -> /Sensor board 4/MCUL_~{RST}
Routing:
- net /Sensor board 1/MCUL_~{RST}: track 0.00 -> 99.2 mm, vias 0 -> 4
- net /SLAVE_~{RST}: track 97.8 -> 0.00 mm, vias 4 -> 0
- net /Sensor board 1/SCL_{1}: track 0.81 -> 82.3 mm, vias 1 -> 5
- net /Sensor board 1/SDA_{2}: track 0.81 -> 77.1 mm, vias 1 -> 5
- net /Sensor board 1/SDA_{1}: track 0.81 -> 77.1 mm, vias 1 -> 5
- net /Sensor board 1/SCL_{2}: track 0.81 -> 67.1 mm, vias 1 -> 5
- net /Sensor board 1/LINE_{2}: track 51.1 -> 104.5 mm, vias 3 -> 4
- net /Sensor board 1/Sensor 2/TRIG_OUT_{5V}: track 47.8 -> 99.4 mm, vias 3 -> 4
- net /Sensor board 1/ADC1_TRIG_OUT: track 38.1 -> 81.4 mm, vias 1 -> 2
- net /Sensor board 1/Sensor 1/TRIG_OUT_{5V}: track 44.7 -> 87.4 mm, vias 3 -> 4
- net /Sensor board 1/ADC3_TRIG_IN: track 0.00 -> 39.6 mm, vias 0 -> 2
- net /Sensor board 1/NDR_{2}: track 47.1 -> 81.0 mm
- net /Sensor board 1/BIN_{2}: track 50.7 -> 81.0 mm
- net /Sensor board 1/ADC3_TRIG_OUT: track 44.1 -> 74.2 mm, vias 1 -> 2
- net /Sensor board 1/CLOCK_{2}: track 51.1 -> 78.3 mm
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