File: bioptics-bx4x4-dc44-camera-board.kicad_pcb (KiCad board)
At the start: 4 copper layers, 260 x 187 mm, 475 parts, among them J1 RadEye1, J10 RadEye1, J11 RadEye1, J12 TagConnect_TC2030_SWD, J13 RadEye1, J14 RadEye1, J2 RadEye1, J3 USB_C_Receptacle_USB2.0, J4 TagConnect_TC2030_SWD, J5 TagConnect_TC2030_SWD, J6 TagConnect_TC2030_SWD, J7 RadEye1, J8 RadEye1, J9 TagConnect_TC2030_SWD, U1 AMS1117-3.3, U10 SRV05-4, U11 IS4xS32160F-xTL, U12 USB3300-EZK, U13 AMS1117-3.3, U14 STM32H753IITx, U15 CJ431, U16 7408, U17 CJ431, U18 AMS1117-3.3, U19 STM32H753IITx, U2 STM32H753IITx, U20 7408, U21 SN74AVC8T245PW, U22 AD5112, U23 INA849, U24 SN74AVC8T245PW, U25 AD5112, U26 INA849, U28 AMS1117-3.3, U29 STM32H753IITx, U3 SN74AVC8T245PW, U30 7408, U31 SN74AVC8T245PW, U32 AD5112, U33 INA849, U34 SN74AVC8T245PW, U35 AD5112, U36 INA849, U38 AMS1117-3.3, U39 STM32H753IITx, U4 AD5112, U40 7408, U41 SN74AVC8T245PW, U42 AD5112, U43 INA849, U44 SN74AVC8T245PW, U45 AD5112, U46 INA849, U5 INA849, U6 SN74AVC8T245PW, U7 AD5112, U8 INA849, U9 FP6291, Y1 24MHz

Commit message: Layout USB connector area
Parts:
- moved R16 424.0 mm to (27.9, 198.2), turned to 90 degrees
- moved R18 408.1 mm to (33.9, 187.2)
- moved R24 404.2 mm to (41.0, 186.8), turned to 90 degrees
- moved C56 404.0 mm to (42.9, 183.1), turned to 90 degrees
- moved C67 395.1 mm to (42.3, 185.3), turned to 180 degrees
- moved R19 394.3 mm to (34.0, 194.0), turned to 180 degrees
- moved C69 390.0 mm to (47.2, 192.7)
- moved R23 386.0 mm to (40.9, 188.2), turned to 180 degrees
- moved C54 383.7 mm to (48.1, 183.1), turned to 90 degrees
- moved C72 379.0 mm to (44.2, 185.3), turned to 180 degrees
- moved R110 378.4 mm to (42.7, 192.6)
- moved C60 378.2 mm to (40.9, 189.5), turned to 180 degrees
- moved C64 377.0 mm to (48.6, 186.1), turned to 90 degrees
- moved Y1 374.8 mm to (45.5, 183.1)
- moved C43 369.9 mm to (25.6, 198.2), turned to 90 degrees
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Routing:
- net +5V: track 77.2 -> 131.8 mm, vias 8 -> 16
- net GND: track 803.3 -> 837.3 mm, vias 214 -> 241
- net Net-(C43-Pad2): track 0.00 -> 21.3 mm
- net /D+: track 0.00 -> 15.7 mm
- net /D-: track 0.00 -> 15.6 mm, vias 0 -> 2
- net Net-(C69-Pad1): track 0.00 -> 11.1 mm, vias 0 -> 2
- net Net-(J5-Pad4): track 96.1 -> 106.8 mm, vias 3 -> 4
- net Net-(J6-Pad4): track 96.1 -> 106.8 mm, vias 3 -> 4
- net Net-(J9-Pad4): track 96.1 -> 106.8 mm, vias 3 -> 4
- net Net-(J12-Pad4): track 96.1 -> 106.8 mm, vias 3 -> 4
- net +3V3: track 0.00 -> 9.30 mm, vias 0 -> 2
- net Net-(C54-Pad2): track 0.00 -> 6.39 mm
- net Net-(C56-Pad1): track 0.00 -> 4.56 mm
- net Net-(J3-PadB5): track 0.00 -> 4.25 mm
- net Net-(J3-PadA5): track 0.00 -> 4.22 mm
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