File: sensor.kicad_sch (KiCad schematic)
At the start: 26 parts

Commit message: Annotate components
Parts:
- gave numbers to parts that had none: 26
Connections:
- net at U22.2 (A): now also U23.3 (Rg); no longer U23.2 (Rg)
- net at U22.3 (W): now also U23.2 (Rg); no longer U23.3 (Rg)

Commit message: Fix shifted FMC D30 and D31 on main STM32
Pins for D30 and D31 were shifted up by one pin
Parts:
- renumbered C122 to C212, C123 to C213, C124 to C214, C125 to C215, C126 to C216, C127 to C217, C128 to C218, C129 to C219, C130 to C220, C131 to C221, FB14 to FB32, FB15 to FB33, FB16 to FB34, J7 to J13, L13 to L25, L14 to L26, R54 to R100, R55 to R101, R56 to R102, R50 to R96, R51 to R97, R52 to R98, R53 to R99, U21 to U41, U22 to U42, U23 to U43

Commit message: Use FC1-15-02-T-WT connector for RadEye1 modules
Parts:
- J11: renamed from J13; symbol Connector_Generic:Conn_01x15 -> Connector_Generic_MountingPin:Conn_01x15_MountingPin
- renumbered C212 to C177, C213 to C178, C214 to C179, C215 to C180, C216 to C181, C217 to C182, C218 to C183, C219 to C184, C220 to C185, C221 to C186, FB32 to FB26, FB33 to FB27, FB34 to FB28, L25 to L21, L26 to L22, R96 to R80, R97 to R81, R98 to R82, R99 to R83, R100 to R84, R101 to R85, R102 to R86, U41 to U34, U42 to U35, U43 to U36
Connections:
- net GND: now also J11.MP (MountPin)

Commit message: First acquisition channel layout WiP
Parts:
- J1: renamed from J11; footprint (none) -> Connector_Samtec_FC1:FC1-15-02-T-WT_P1.0mm
- renumbered C177 to C23, C178 to C24, C179 to C25, C180 to C26, C181 to C27, C182 to C28, C183 to C29, C184 to C30, C185 to C31, C186 to C32, FB26 to FB2, FB27 to FB3, FB28 to FB4, L21 to L2, L22 to L3, R80 to R2, R81 to R3, R82 to R4, R83 to R5, R84 to R6, R85 to R7, R86 to R8, U34 to U3, U35 to U4, U36 to U5
Connections:
- net BIN: now also U3.17 (B5); no longer U3.18 (B4)
- net BIN_{5V}: now also U3.7 (A5); no longer U3.6 (A4)
- net CLOCK: now also U3.16 (B6); no longer U3.19 (B3)
- net CLOCK_{5V}: now also U3.8 (A6); no longer U3.5 (A3)
- net GND: now also U3.20 (B2), U3.21 (B1); no longer U3.14 (B8), U3.15 (B7)
- net NDR: now also U3.18 (B4); no longer U3.17 (B5)
- net NDR_{5V}: now also U3.6 (A4); no longer U3.7 (A5)
- net RESET: now also U3.14 (B8); no longer U3.21 (B1)
- net RESET_{5V}: now also U3.10 (A8); no longer U3.3 (A1)
- net START: now also U3.15 (B7); no longer U3.20 (B2)
- net START_{5V}: now also U3.9 (A7); no longer U3.4 (A2)
- net TRIG_IN_{3V3}: now also U3.19 (B3); no longer U3.16 (B6)
- net TRIG_OUT_{5V}: now also U3.5 (A3); no longer U3.8 (A6)
- net at U4.2 (A): now also U5.2 (Rg); no longer U5.3 (Rg)
- net at U4.3 (W): now also U5.3 (Rg); no longer U5.2 (Rg)

Commit message: Decouple MCU resets via diode
Parts:
- renumbered C23 to C222, C24 to C223, C25 to C224, C26 to C225, C27 to C226, C28 to C227, C29 to C228, C30 to C229, C31 to C230, C32 to C231, FB2 to FB35, FB3 to FB36, FB4 to FB37, J1 to J14, L2 to L27, L3 to L28, R2 to R103, R3 to R104, R4 to R105, R5 to R106, R6 to R107, R7 to R108, R8 to R109, U3 to U44, U4 to U45, U5 to U46
Connections:
- net BIN: now also U44.18 (B4); no longer U44.17 (B5)
- net BIN_{5V}: now also U44.6 (A4); no longer U44.7 (A5)
- net CLOCK: now also U44.19 (B3); no longer U44.16 (B6)
- net CLOCK_{5V}: now also U44.5 (A3); no longer U44.8 (A6)
- net GND: now also U44.14 (B8), U44.15 (B7); no longer U44.20 (B2), U44.21 (B1)
- net NDR: now also U44.17 (B5); no longer U44.18 (B4)
- net NDR_{5V}: now also U44.7 (A5); no longer U44.6 (A4)
- net RESET: now also U44.21 (B1); no longer U44.14 (B8)
- net RESET_{5V}: now also U44.3 (A1); no longer U44.10 (A8)
- net START: now also U44.20 (B2); no longer U44.15 (B7)
- net START_{5V}: now also U44.4 (A2); no longer U44.9 (A7)
- net TRIG_IN_{3V3}: now also U44.16 (B6); no longer U44.19 (B3)
- net TRIG_OUT_{5V}: now also U44.8 (A6); no longer U44.5 (A3)

Commit message: Use two instead of four 3.8V voltage references
Parts:
- renumbered C222 to C23, C223 to C24, C224 to C25, C225 to C26, C226 to C27, C227 to C28, C228 to C29, C229 to C30, C230 to C31, C231 to C32, FB35 to FB2, FB36 to FB3, FB37 to FB4, J14 to J1, L27 to L2, L28 to L3, R103 to R2, R104 to R3, R105 to R4, R106 to R5, R107 to R6, R108 to R7, R109 to R8, U44 to U3, U45 to U4, U46 to U5

Commit message: Add sensor board power planes
Parts:
- renumbered C23 to C222, C24 to C223, C25 to C224, C26 to C225, C27 to C226, C28 to C227, C29 to C228, C30 to C229, C31 to C230, C32 to C231, FB2 to FB35, FB3 to FB36, FB4 to FB37, J1 to J14, L2 to L27, L3 to L28, R2 to R103, R3 to R104, R4 to R105, R5 to R106, R6 to R107, R7 to R108, R8 to R109, U3 to U44, U4 to U45, U5 to U46
